File: kezfertotlenito.sch (KiCad schematic (older format))
At the start: 33 parts, among them M1 A1150, Q1 BC556, Q2 BC547, Q3 IRF9540N, U1 TLC2252, U2 TLC2252

Commit message: Proto NYÁK
Parts:
- BT1, M1: footprint (none) -> Connector_PinHeader_2.54mm:PinHeader_1x02_P2.54mm_Vertical
- C1, C2, C4, C6: footprint (none) -> Capacitor_SMD:C_1206_3216Metric_Pad1.33x1.80mm_HandSolder
- C3, C5, C7: footprint (none) -> Capacitor_THT:CP_Radial_D6.3mm_P2.50mm
- D1: footprint (none) -> Diode_SMD:D_MELF
- D3, D4: footprint (none) -> LED_THT:LED_D5.0mm
- F1: footprint (none) -> Fuse:Fuseholder_Cylinder-5x20mm_Stelvio-Kontek_PTF78_Horizontal_Open
- R1, R10, R11, R12, R2, R3, R4, R5, R6, R7, R8, R9: footprint (none) -> Resistor_SMD:R_1206_3216Metric_Pad1.30x1.75mm_HandSolder
- U1, U2: footprint (none) -> Package_SO:SOIC-8_3.9x4.9mm_P1.27mm
Connections:
- net +6V: now also D4.1 (K)
- net -6V: no longer D4.2 (A)
- net GND: now also U2.5 (+); no longer U1.5 (+)
- net at C4.2, R7.1: now also D4.2 (A), U2.6 (-); no longer D4.1 (K), U1.6 (-)
- net at C4.1, Q1.2 (B), R7.2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: now also U2.7; no longer U1.7
- net at C6.1, D5.1 (K), R10.2: now also U1.5 (+); no longer U2.5 (+)
- net at Q2.1 (C), R11.2, R12.1: now also U1.6 (-); no longer U2.6 (-)
- net at Q3.1 (G), R10.1, R11.1: now also U1.7; no longer U2.7
Other:
- note added: "Kiss Ádám és Illés Tibor, SEM"
- note removed: "Kiss Ádám, SEM"
- moved on the sheet: D4, U1B, U2B
